Commit message: change initial arm pose

File: urdf/braccio_arm.urdf (robot description, URDF)
Before this commit: robot visual, 8 links, 7 joints
Joints:
- joint elbow_joint: origin xyz=0 0 0.125 rpy=-1.5708 0 0 -> xyz=0 0 0.125 rpy=-0.5 0 0
- joint shoulder_joint: origin xyz=0 -0.002 0.072 rpy=-1.5708 0 0 -> xyz=0 -0.002 0.072 rpy=-1.0 0 0

Commit message: Update URDF model

File: urdf/braccio_arm.urdf (robot description, URDF)
Before this commit: robot visual, 8 links, 7 joints
Joints:
- joint elbow_joint: origin xyz=0 0 0.125 rpy=-0.5 0 0 -> xyz=0 0 0.125 rpy=-1.5708 0 0
- joint shoulder_joint: origin xyz=0 -0.002 0.072 rpy=-1.0 0 0 -> xyz=0 -0.002 0.072 rpy=-1.5708 0 0

Commit message: Renaming package

File: urdf/braccio_arm.urdf (robot description, URDF)
Before this commit: robot visual, 8 links, 7 joints
Links:
- link braccio_base_link: geometry visual mesh filename=package://braccio_camai/meshes/braccio_base.stl scale=0.001 0.001 0.001
- link elbow_link: geometry visual mesh filename=package://braccio_camai/meshes/braccio_elbow.stl scale=0.001 0.001 0.001
- link left_gripper_link: geometry visual mesh filename=package://braccio_camai/meshes/braccio_left_gripper.stl scale=0.001 0.001 0.001
- link right_gripper_link: geometry visual mesh filename=package://braccio_camai/meshes/braccio_right_gripper.stl scale=0.001 0.001 0.001
- link shoulder_link: geometry visual mesh filename=package://braccio_camai/meshes/braccio_shoulder.stl scale=0.001 0.001 0.001
- link wrist_pitch_link: geometry visual mesh filename=package://braccio_camai/meshes/braccio_wrist_pitch.stl scale=0.001 0.001 0.001
- link wrist_roll_link: geometry visual mesh filename=package://braccio_camai/meshes/braccio_wrist_roll.stl scale=0.001 0.001 0.001
